File: Buck/Buck.kicad_pcb (KiCad board)
At the start: 2 copper layers, 86.8 x 45.7 mm, 32 parts, among them IC1 LM5148RGYR

Commit message: Updated
Parts:
- removed H1, H2, H3, H4: MountingHole, MountingHole:MountingHole_2.1mm
- removed IC1: LM5148RGYR, LM5148_:LM5148RGYR
- added IC3: LM5148RGYR, LM5148_:LM5148RGYR, F.Cu at (141.5, 123.0)
- NT1: moved to F.Cu
- moved C2 5.46 mm to (144.6, 118.0)
- moved C3 5.46 mm to (144.6, 113.2)
- moved C4 5.13 mm to (150.8, 109.3)
- moved Q1 5.13 mm to (150.9, 115.7)
- moved Q2 5.13 mm to (150.8, 124.3)
- moved R6 3.35 mm to (140.3, 118.3), turned to 90 degrees
- moved L1 2.83 mm to (169.8, 122.8)
- moved NT1 2.76 mm to (143.2, 123.8), turned to -90 degrees
- moved C9 2.71 mm to (146.7, 124.9), turned to -90 degrees
- moved C13 2.55 mm to (187.0, 135.8)
- moved C12 2.40 mm to (187.0, 130.9)
- moved R7 2.40 mm to (187.1, 123.0), turned to 90 degrees
- moved C10 2.25 mm to (187.0, 109.5)
- moved C11 2.25 mm to (187.0, 115.0)
- moved R1 1.73 mm to (133.7, 135.7)
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Connections:
- C1 pad 1: VIN -> GND
- C1 pad 2: GND -> VIN
- C2 pad 1: VIN -> GND
- C2 pad 2: GND -> VIN
- C3 pad 1: VIN -> GND
- C3 pad 2: GND -> VIN
- C4 pad 1: VIN -> GND
- C4 pad 2: GND -> VIN
- C7 pad 1: VDDA -> GND2
- C7 pad 2: GND2 -> Net-(IC3-PFM/SYNC)
- C8 pad 1: VCC -> Net-(IC3-VCC)
- C9 pad 1: Net-(IC1-CBOOT) -> Net-(IC3-SW)
- C9 pad 2: Net-(IC1-SW) -> Net-(IC3-CBOOT)
- L1 pad 2: Net-(IC1-SW) -> Net-(IC3-SW)
- Q1 pad 1: Net-(IC1-SW) -> Net-(IC3-SW)
- Q1 pad 2: Net-(IC1-SW) -> Net-(IC3-HO)
- Q1 pad 3: Net-(IC1-SW) -> VIN
- Q1 pad 4: HO -> (no net)
- Q1 pad 5: VIN -> (no net)
- Q1 pad 6: VIN -> (no net)
- Q1 pad 7: VIN -> (no net)
- Q1 pad 8: VIN -> (no net)
- Q2 pad 2: GND -> Net-(IC3-LO)
- Q2 pad 3: GND -> Net-(IC3-SW)
- Q2 pad 4: GND -> (no net)
- Q2 pad 5: Net-(IC1-SW) -> (no net)
- Q2 pad 6: Net-(IC1-SW) -> (no net)
- Q2 pad 7: Net-(IC1-SW) -> (no net)
- Q2 pad 8: Net-(IC1-SW) -> (no net)
- R3 pad 1: VDDA -> Net-(IC3-FB)
- R3 pad 2: Net-(IC1-FB) -> Net-(IC3-PFM/SYNC)
- R4 pad 1: GND2 -> Net-(IC3-RT)
- R4 pad 2: Net-(IC1-RT) -> GND2
- R5 pad 1: GND2 -> Net-(IC3-CNFG)
- R5 pad 2: Net-(IC1-CNFG) -> GND2
- R6 pad 1: Net-(IC1-PG/SYNCOUT) -> Net-(IC3-VCC)
- R6 pad 2: VCC -> Net-(IC3-PG/SYNCOUT)
Other:
- board size 86.8 x 45.7 mm -> 82.3 x 47.9 mm

Commit message: updated
Parts:
- removed U1, U2: ~, pad_footprint:Untitled
- added H1: MountingHole, MountingHole:MountingHole_2.1mm, F.Cu at (105.6, 99.2)
- added H2: MountingHole, MountingHole:MountingHole_2.1mm, F.Cu at (105.6, 104.9)
- added H3: MountingHole, MountingHole:MountingHole_2.1mm, F.Cu at (105.6, 110.7)
- added H4: MountingHole, MountingHole:MountingHole_2.1mm, F.Cu at (105.6, 116.4)
- added J1: Conn_01x02, Connector_Samtec_MicroPower:Samtec_UMPS-02-XX.X-X-V-S_1x02_P2.0mm_Socket, F.Cu at (121.5, 123.2)
- added J2: Conn_01x02, Connector_Samtec_MicroPower:Samtec_UMPS-02-XX.X-X-V-S_1x02_P2.0mm_Socket, F.Cu at (200.9, 122.8)
- C5: value 4.7uf -> 4.7nf
- Q1, Q2: value ~ -> CSD18534Q5A; footprint CSD18534Q5A:Q5A -> CSD18534Q5A_:NEW
Other:
- board size 82.3 x 47.9 mm -> 89.8 x 47.9 mm

Commit message: .updated
Parts:
- J1, J2: footprint Connector_Samtec_MicroPower:Samtec_UMPS-02-XX.X-X-V-S_1x02_P2.0mm_Socket -> pad_footprint:Untitled
- moved J2 2.46 mm to (198.4, 122.9), turned to 0 degrees
- moved R7 1.02 mm to (188.1, 123.1)
- moved J1 0.48 mm to (121.8, 122.9), turned to 0 degrees
- turned C4 to 0 degrees
Routing:
- net GND: track 0.00 -> 180.8 mm, vias 0 -> 71
- net VOUT: track 0.00 -> 114.1 mm, vias 0 -> 26
- net VIN: track 0.00 -> 84.7 mm, vias 0 -> 2
- net ISNS: track 0.00 -> 64.7 mm, vias 0 -> 2
- net Net-(IC3-SW): track 0.00 -> 46.2 mm
- net GND2: track 0.00 -> 31.2 mm, vias 0 -> 2
- net Net-(IC3-PFM/SYNC): track 0.00 -> 21.3 mm, vias 0 -> 2
- net Net-(IC3-VCC): track 0.00 -> 18.3 mm, vias 0 -> 2
- net Net-(IC3-LO): track 0.00 -> 13.2 mm
- net Net-(IC3-HO): track 0.00 -> 11.3 mm, vias 0 -> 2
- net Net-(IC3-EXTCOMP): track 0.00 -> 9.03 mm
- net Net-(IC3-CBOOT): track 0.00 -> 7.71 mm, vias 0 -> 2
- net Net-(IC3-RT): track 0.00 -> 5.50 mm
- net Net-(IC3-CNFG): track 0.00 -> 5.49 mm
- net Net-(IC3-FB): track 0.00 -> 5.48 mm
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- added copper zone on B.Cu, net GND
- added copper zone on F.Cu, net GND
- added copper zone on F.Cu, net GND2
- added copper zone on F.Cu, net Net-(IC3-SW)
- added copper zone on F.Cu, net VOUT
Other:
- board size 89.8 x 47.9 mm -> 82.8 x 47.9 mm

Commit message: UPDATED
Parts:
- removed IC3: LM5148RGYR, LM5148_:LM5148RGYR
- added IC1: LM5148RGYR, LM5148_:LM5148RGYR, F.Cu at (141.5, 123.0)
- moved H3 98.3 mm to (198.4, 143.2)
- moved H2 92.9 mm to (198.5, 102.9)
- moved H4 32.2 mm to (123.9, 142.9)
- moved LED1 31.1 mm to (131.4, 107.4), turned to -90 degrees
- moved R1 23.3 mm to (131.5, 112.6), turned to 90 degrees
- moved C1 21.7 mm to (144.6, 109.0), turned to 0 degrees
- moved H1 18.6 mm to (123.9, 102.9)
- moved C8 14.2 mm to (138.7, 116.8), turned to 90 degrees
- moved C9 5.69 mm to (144.9, 119.5), turned to 180 degrees
- moved C7 2.85 mm to (140.9, 129.2)
- moved R3 2.15 mm to (140.4, 127.5), turned to 0 degrees
- moved C2 1.73 mm to (144.6, 116.3), turned to 0 degrees
- moved NT1 1.67 mm to (141.7, 123.3), turned to 90 degrees
- moved R6 1.51 mm to (140.3, 116.8)
- moved R7 1.25 mm to (187.0, 123.6), turned to 0 degrees
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Routing:
- net VIN: track 84.7 -> 116.3 mm
- net GND: track 180.8 -> 155.8 mm, vias 71 -> 98
- net Net-(IC1-LO): track 13.2 -> 19.0 mm
- net Net-(IC1-CBOOT): track 7.71 -> 2.40 mm, vias 2 -> 0
- net GND2: track 31.2 -> 26.6 mm
- net Net-(IC1-SW): track 46.2 -> 42.3 mm
- net Net-(IC1-PFM/SYNC): track 21.3 -> 23.8 mm
- net Net-(IC1-FB): track 5.48 -> 3.35 mm
- net VOUT: track 114.1 -> 115.9 mm, vias 26 -> 2
- net ISNS: track 64.7 -> 66.3 mm
- net Net-(IC1-PG/SYNCOUT): track 5.24 -> 6.54 mm
- net Net-(IC1-EXTCOMP): track 9.03 -> 8.39 mm
