File: Buck/Buck.kicad_pcb (KiCad board)
At the start: 2 copper layers, 82.8 x 47.9 mm, 32 parts, among them IC1 LM5148RGYR, J1 Conn_01x02, J2 Conn_01x02, Q1 CSD18534Q5A, Q2 CSD18534Q5A

Commit message: logo added
added the logo
Parts:
- added G***: LOGO, Logo:BoltzRndLogo10mm, F.Cu at (192.3, 140.5)
Other:
- board text added: "2-12S Buck Converter"
- board text added: "Boltz R&D"
- board text added: "www.boltzrnd.com"
