File: Buck/Buck.kicad_sch (KiCad schematic)
At the start: 32 parts, among them IC1 LM5148RGYR

Commit message: Updated
Parts:
- removed IC1: LM5148RGYR, LM5148_:LM5148RGYR, symbol LM5148RGYR:LM5148RGYR
- added IC3: LM5148RGYR, LM5148RGYR, symbol LM5148RGYR_edited normal_symbol:LM5148RGYR
Connections:
- net GND: now also C1.1, C2.1, C3.1, C4.1, IC3.1 (NC_1), IC3.10 (PGND), IC3.16 (VCCX), IC3.2 (NC_2), IC3.22 (NC_3), IC3.23 (NC_4), IC3.24 (NC_5); no longer C1.2, C2.2, C3.2, C4.2
- net GND2: now also C7.1, R4.2, R5.2, IC3.25 (AGND_2), IC3.7 (AGND_1); no longer C7.2, R4.1, R5.1
- net ISNS: now also IC3.20 (ISNS+)
- net VIN: now also C1.2, C2.2, C3.2, C4.2, IC3.12 (VIN), IC3.19 (EN); no longer C1.1, C2.1, C3.1, C4.1
- net VOUT: now also IC3.21 (VOUT)
- net at L1.2, Q1.1 (S), Q2.3 (D): now also C9.1, IC3.14 (SW); no longer C9.2
- net at R6.1: now also C8.1, IC3.9 (VCC)
- net at C6.1, R2.2: now also IC3.5 (EXTCOMP)
- net at R3.2: now also C7.2, IC3.18 (PFM/SYNC), IC3.8 (VDDA)
- net HO: no longer names the net of Q1.2 (G)
- net HO: now also IC3.13 (HO)
- net LO: no longer names the net of Q2.2 (G)
- net LO: now also IC3.11 (LO)
- net VCC: no longer names the net of R6.2
- net VCC: now also IC3.17 (PG/SYNCOUT); no longer C8.1
- net VDDA: no longer names the net of R3.1
- net VDDA: now also IC3.6 (FB); no longer C7.1
- new net: C9.2, IC3.15 (CBOOT)
- new net: IC3.3 (CNFG), R5.1
- new net: IC3.4 (RT), R4.1
Other:
- moved on the sheet: C1, C10, C11, C12, C13, C2, C3, C4, C5, C6, C7, C8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

Commit message: updated
Parts:
- removed U1: ~, pad_footprint:Untitled, symbol input_pad:I/P
- removed U2: ~, pad_footprint:Untitled, symbol output_pad:o/p
- added J1, J2: Conn_01x02, Connector_Samtec_MicroPower:Samtec_UMPS-02-XX.X-X-V-S_1x02_P2.0mm_Socket, symbol Connector_Generic:Conn_01x02
- C5: value 4.7uf -> 4.7nf
- H1, H2, H3, H4, NT1: now in the parts list
- IC3: footprint LM5148RGYR -> LM5148_:LM5148RGYR
- Q1, Q2: value ~ -> CSD18534Q5A; footprint CSD18534Q5A:Q5A -> CSD18534Q5A_:NEW
Connections:
- net GND: now also J1.2 (Pin_2), J2.2 (Pin_2)
- net VIN: now also J1.1 (Pin_1)
- net VOUT: now also J2.1 (Pin_1)
Changed lines of the file:
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@@
 		(fields_autoplaced yes)
 		(property "Reference" "Q1"
-			(at 212.09 74.2949 0)
+			(at 212.09 73.6599 0)
 			(effects
 				(font
@@
 			)
 		)
-		(property "Value" "~"
-			(at 212.09 76.2 0)
+		(property "Value" "CSD18534Q5A"
+			(at 212.09 76.1999 0)
 			(effects
 				(font
@@
 			)
 		)
-		(property "Footprint" "CSD18534Q5A:Q5A"
+		(property "Footprint" "CSD18534Q5A_:NEW"
 			(at 210.82 76.835 0)
 			(effects
@@
 		(unit 1)
 		(exclude_from_sim yes)
-		(in_bom no)
+		(in_bom yes)
 		(on_board yes)
 		(dnp no)
@@
 			)
 		)
-		(property "Value" "~"
+		(property "Value" "CSD18534Q5A"
 			(at 212.09 113.03 0)
 			(effects
@@
 			)
 		)
-		(property "Footprint" "CSD18534Q5A:Q5A"
+		(property "Footprint" "CSD18534Q5A_:NEW"
 			(at 210.82 113.665 0)
 			(effects
@@
 		(unit 1)
 		(exclude_from_sim yes)
-		(in_bom no)
+		(in_bom yes)
 		(on_board yes)
 		(dnp no)
@@
 			)
 		)
-		(property "Footprint" "LM5148RGYR"
+		(property "Footprint" "LM5148_:LM5148RGYR"
 			(at 138.176 84.074 0)
 			(effects
@@
 		(unit 1)
 		(exclude_from_sim yes)
-		(in_bom no)
+		(in_bom yes)
 		(on_board yes)
 		(dnp no)
@@
 		(unit 1)
 		(exclude_from_sim no)
-		(in_bom no)
+		(in_bom yes)
 		(on_board yes)
 		(dnp no)
@@
 	)
 	(symbol
-		(lib_id "Device:C")
-		(at 161.29 160.02 180)
+		(lib_id "Connector_Generic:Conn_01x02")
+		(at 186.69 24.13 0)
 		(unit 1)
 		(exclude_from_sim no)
@@
 		(dnp no)
 		(fields_autoplaced yes)
-		(property "Reference" "C1"
-			(at 157.48 161.2901 0)
+		(property "Reference" "J1"
+			(at 189.23 24.1299 0)
 			(effects
 				(font
@@
 			)
 		)
-		(property "Value" "4.7uf"
-			(at 157.48 158.7501 0)
+		(property "Value" "Conn_01x02"
+			(at 189.23 26.6699 0)
 			(effects
 				(font
@@
 				)
 				(justify left)
-			)
-		)
-		(property "Footprint" "Capacitor_SMD:C_1210_3225Metric"
-			(at 160.3248 156.21 0)
-			(effects
-				(font
-					(size 1.27 1.27)
-				)
 				(hide yes)
 			)
 		)
-		(property "Datasheet" "~"
-			(at 161.29 160.02 0)
+		(property "Footprint" "Connector_Samtec_MicroPower:Samtec_UMPS-02-XX.X-X-V-S_1x02_P2.0mm_Socket"
+			(at 186.69 24.13 0)
 			(effects
 				(font
@@
 			)
 		)
-		(property "Description" "Unpolarized capacitor"
-			(at 161.29 160.02 0)
-			(effects
-				(font
-					(size 1.27 1.27)
-				)
-				(hide yes)
-			)
-		)
-		(property "mfg no" "FS32X475K101EGG"
-			(at 161.29 160.02 0)
+		(property "Datasheet" "~"
+			(at 186.69 24.13 0)
 			(effects
 				(font
@@
 			)
 		)
-		(property "LCSC NO" "C381466"
-			(at 161.29 160.02 0)
+		(property "Description" "Generic connector, single row, 01x02, script generated (kicad-library-utils/schlib/autogen/connector/)"
+			(at 186.69 24.13 0)
 			(effects
 				(font
@@
 			(project ""
 				(path "/2b20bf84-f1a7-4c48-aa1b-8d85c83ac6e5"
-					(reference "C1")
+					(reference "J1")
 					(unit 1)
 				)
@@
 	)
 	(symbol
-		(lib_id "Device:R")
-		(at 104.14 123.19 0)
+		(lib_id "Device:C")
+		(at 161.29 160.02 180)
 		(unit 1)
 		(exclude_from_sim no)
@@
 		(dnp no)
 		(fields_autoplaced yes)
-		(property "Reference" "R5"
-			(at 106.68 121.9199 0)
+		(property "Reference" "C1"
+			(at 157.48 161.2901 0)
 			(effects
 				(font
@@
 			)
 		)
-		(property "Value" "40.2kohm"
-			(at 106.68 124.4599 0)
+		(property "Value" "4.7uf"
+			(at 157.48 158.7501 0)
 			(effects
 				(font
@@
 			)
 		)
-		(property "Footprint" "Capacitor_SMD:C_0603_1608Metric"
-			(at 102.362 123.19 90)
+		(property "Footprint" "Capacitor_SMD:C_1210_3225Metric"
+			(at 160.3248 156.21 0)
 			(effects
 				(font
@@
 		)
 		(property "Datasheet" "~"
-			(at 104.14 123.19 0)
+			(at 161.29 160.02 0)
 			(effects
 				(font
@@
 			)
 		)
-		(property "Description" "Resistor"
-			(at 104.14 123.19 0)
+		(property "Description" "Unpolarized capacitor"
+			(at 161.29 160.02 0)
 			(effects
 				(font
@@
 			)
 		)
-		(property "MFG NO" "CRCW060340K2FKEA"
-			(at 104.14 123.19 0)
+		(property "mfg no" "FS32X475K101EGG"
+			(at 161.29 160.02 0)
 			(effects
 				(font
@@
 			)
 		)
-		(property "LCSC NO" "C844784"
-			(at 104.14 123.19 0)
+		(property "LCSC NO" "C381466"
+			(at 161.29 160.02 0)
 			(effects
 				(font
@@
 			(project ""
 				(path "/2b20bf84-f1a7-4c48-aa1b-8d85c83ac6e5"
-					(reference "R5")
+					(reference "C1")
 					(unit 1)
 				)
@@
 	)
 	(symbol
-		(lib_id "input_pad:I/P")
-		(at 181.61 25.4 0)
+		(lib_id "Device:R")
+		(at 104.14 123.19 0)
 		(unit 1)
 		(exclude_from_sim no)
@@
 		(dnp no)
 		(fields_autoplaced yes)
-		(property "Reference" "U1"
-			(at 190.5 24.7649 0)
+		(property "Reference" "R5"
+			(at 106.68 121.9199 0)
 			(effects
 				(font
@@
 			)
 		)
-		(property "Value" "~"
-			(at 190.5 26.67 0)
+		(property "Value" "40.2kohm"
+			(at 106.68 124.4599 0)
 			(effects
 				(font
@@
 			)
 		)
-		(property "Footprint" "pad_footprint:Untitled"
-			(at 181.61 25.4 0)
+		(property "Footprint" "Capacitor_SMD:C_0603_1608Metric"
+			(at 102.362 123.19 90)
 			(effects
 				(font
@@
 			)
 		)
-		(property "Datasheet" ""
-			(at 181.61 25.4 0)
+		(property "Datasheet" "~"
+			(at 104.14 123.19 0)
+			(effects
+				(font
+					(size 1.27 1.27)
+				)
+				(hide yes)
+			)
+		)
+		(property "Description" "Resistor"
+			(at 104.14 123.19 0)
 			(effects
 				(font
@@
 			)
 		)
-		(property "Description" ""
-			(at 181.61 25.4 0)
+		(property "MFG NO" "CRCW060340K2FKEA"
+			(at 104.14 123.19 0)
 			(effects
 				(font
@@
 			)
 		)
-		(pin "2"
+		(property "LCSC NO" "C844784"
+			(at 104.14 123.19 0)
+			(effects
+				(font
+					(size 1.27 1.27)
+				)
+				(hide yes)
+			)
 		)
 		(pin "1"
 		)
+		(pin "2"
+		)
 		(instances
 			(project ""
 				(path "/2b20bf84-f1a7-4c48-aa1b-8d85c83ac6e5"
-					(reference "U1")
+					(reference "R5")
 					(unit 1)
 				)
@@
 	)
 	(symbol
-		(lib_id "output_pad:o/p")
-		(at 204.47 25.4 0)
-		(unit 1)
-		(exclude_from_sim no)
-		(in_bom yes)
-		(on_board yes)
-		(dnp no)
-		(fields_autoplaced yes)
-		(property "Reference" "U2"
-			(at 213.36 24.7649 0)
-			(effects
-				(font
-					(size 1.27 1.27)
-				)
-				(justify left)
-			)
-		)
-		(property "Value" "~"
-			(at 213.36 26.67 0)
-			(effects
-				(font
-					(size 1.27 1.27)
-				)
-				(justify left)
-			)
-		)
-		(property "Footprint" "pad_footprint:Untitled"
-			(at 204.47 25.4 0)
-			(effects
-				(font
-					(size 1.27 1.27)
-				)
-				(hide yes)
-			)
-		)
-		(property "Datasheet" ""
-			(at 204.47 25.4 0)
-			(effects
-				(font
-					(size 1.27 1.27)
-				)
-				(hide yes)
-			)
-		)
-		(property "Description" ""
-			(at 204.47 25.4 0)
-			(effects
-				(font
-					(size 1.27 1.27)
-				)
-				(hide yes)
-			)
-		)
-		(pin "1"
-		)
-		(pin "2"
-		)
-		(instances
-			(project ""
-				(path "/2b20bf84-f1a7-4c48-aa1b-8d85c83ac6e5"
-					(reference "U2")
-					(unit 1)
-				)
-			)
-		)
-	)
-	(symbol
 		(lib_id "power:GND")
 		(at 274.32 31.75 0)
@@
 			)
 		)
-		(property "Value" "4.7uf"
+		(property "Value" "4.7nf"
 			(at 60.96 118.11 90)
 			(effects
@@
 		(unit 1)
 		(exclude_from_sim yes)
-		(in_bom no)
+		(in_bom yes)
 		(on_board yes)
 		(dnp no)
@@
 					(unit 1)
 				)
+			)
+		)
+	)
+	(symbol
+		(lib_id "Connector_Generic:Conn_01x02")
+		(at 209.55 24.13 0)
+		(unit 1)
+		(exclude_from_sim no)
+		(in_bom yes)
+		(on_board yes)
+		(dnp no)
+		(fields_autoplaced yes)
+		(property "Reference" "J2"
+			(at 212.09 24.1299 0)
+			(effects
+				(font
+					(size 1.27 1.27)
+				)
+				(justify left)
+			)
+		)
+		(property "Value" "Conn_01x02"
+			(at 212.09 26.6699 0)
+			(effects
+				(font
+					(size 1.27 1.27)
+				)
+				(justify left)
+				(hide yes)
+			)
+		)
+		(property "Footprint" "Connector_Samtec_MicroPower:Samtec_UMPS-02-XX.X-X-V-S_1x02_P2.0mm_Socket"
+			(at 209.55 24.13 0)
+			(effects
+				(font
+					(size 1.27 1.27)
+				)
+				(hide yes)
+			)
+		)
+		(property "Datasheet" "~"
+			(at 209.55 24.13 0)
+			(effects
+				(font
+					(size 1.27 1.27)
+				)
+				(hide yes)
+			)
+		)
+		(property "Description" "Generic connector, single row, 01x02, script generated (kicad-library-utils/schlib/autogen/connector/)"
+			(at 209.55 24.13 0)
+			(effects
+				(font
+					(size 1.27 1.27)
+				)
+				(hide yes)
+			)
+		)
+		(pin "1"
+		)
+		(pin "2"
+		)
+		(instances
+			(project ""
+				(path "/2b20bf84-f1a7-4c48-aa1b-8d85c83ac6e5"
+					(reference "J2")
+					(unit 1)
+				)

Commit message: .updated
Parts:
- J1, J2: footprint Connector_Samtec_MicroPower:Samtec_UMPS-02-XX.X-X-V-S_1x02_P2.0mm_Socket -> pad_footprint:Untitled
Changed lines of the file:
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@@
 			)
 		)
-		(property "Footprint" "Connector_Samtec_MicroPower:Samtec_UMPS-02-XX.X-X-V-S_1x02_P2.0mm_Socket"
+		(property "Footprint" "pad_footprint:Untitled"
 			(at 186.69 24.13 0)
 			(effects
@@
 			)
 		)
-		(property "Footprint" "Connector_Samtec_MicroPower:Samtec_UMPS-02-XX.X-X-V-S_1x02_P2.0mm_Socket"
+		(property "Footprint" "pad_footprint:Untitled"
 			(at 209.55 24.13 0)
 			(effects

Commit message: UPDATED
Parts:
- removed IC3: LM5148RGYR, LM5148_:LM5148RGYR, symbol LM5148RGYR_edited normal_symbol:LM5148RGYR
- added IC1: LM5148RGYR, LM5148_:LM5148RGYR, symbol LM5148RGYR_edited normal_symbol:LM5148RGYR
Connections:
- net GND: now also IC1.1 (NC_1), IC1.10 (PGND), IC1.16 (VCCX), IC1.2 (NC_2), IC1.22 (NC_3), IC1.23 (NC_4), IC1.24 (NC_5), IC1.25 (AGND_2)
- net GND2: now also IC1.7 (AGND_1)
- net ISNS: now also IC1.20 (ISNS+)
- net VIN: now also IC1.12 (VIN), IC1.19 (EN)
- net VOUT: now also IC1.21 (VOUT)
- net at C9.1, L1.2, Q1.1 (S)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: now also IC1.14 (SW)
- net at Q1.2 (G): now also IC1.13 (HO)
- net at C7.2, R3.2: now also IC1.18 (PFM/SYNC), IC1.8 (VDDA)
- net at C6.1, R2.2: now also IC1.5 (EXTCOMP)
- net at Q2.2 (G): now also IC1.11 (LO)
- net at C9.2: now also IC1.15 (CBOOT)
- net at R6.2: now also IC1.17 (PG/SYNCOUT)
- net at R5.1: now also IC1.3 (CNFG)
- net at R4.1: now also IC1.4 (RT)
- net at R3.1: now also IC1.6 (FB)
- net at C8.1, R6.1: now also IC1.9 (VCC)
Changed lines of the file:
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@@
+	)
+	(symbol
+		(lib_id "LM5148RGYR_edited normal_symbol:LM5148RGYR")
+		(at 123.19 95.25 0)
+		(unit 1)
+		(exclude_from_sim no)
+		(in_bom yes)
+		(on_board yes)
+		(dnp no)
+		(fields_autoplaced yes)
+		(property "Reference" "IC1"
+			(at 143.51 77.47 0)
+			(effects
+				(font
+					(size 1.27 1.27)
+				)
+			)
+		)
+		(property "Value" "LM5148RGYR"
+			(at 143.51 80.01 0)
+			(effects
+				(font
+					(size 1.27 1.27)
+				)
+			)
+		)
+		(property "Footprint" "LM5148_:LM5148RGYR"
+			(at 138.176 84.074 0)
+			(effects
+				(font
+					(size 1.27 1.27)
+				)
+				(justify left)
+				(hide yes)
+			)
+		)
+		(property "Datasheet" "https://www.ti.com/lit/ds/symlink/lm5148.pdf?ts=1680990210570&ref_url=https%253A%252F%252Fwww.ti.com%252Fproduct%252FLM5148"
+			(at 171.958 74.676 0)
+			(effects
+				(font
+					(size 1.27 1.27)
+				)
+				(justify left)
+				(hide yes)
+			)
+		)
+		(property "Description" "Switching Controllers 3.5-V to 80-V, current mode synchronous buck controller"
+			(at 100.33 116.84 0)
+			(effects
+				(font
+					(size 1.27 1.27)
+				)
+				(hide yes)
+			)
+		)
+		(property "Description_1" "Switching Controllers 3.5-V to 80-V, current mode synchronous buck controller"
+			(at 171.958 77.216 0)
+			(effects
+				(font
+					(size 1.27 1.27)
+				)
+				(justify left)
+				(hide yes)
+			)
+		)
+		(property "Height" "1"
+			(at 160.02 90.17 0)
+			(effects
+				(font
+					(size 1.27 1.27)
+				)
+				(justify left)
+				(hide yes)
+			)
+		)
+		(property "Manufacturer_Name" "Texas Instruments"
+			(at 172.72 106.68 0)
+			(effects
+				(font
+					(size 1.27 1.27)
+				)
+				(justify left)
+				(hide yes)
+			)
+		)
+		(property "Manufacturer_Part_Number" "LM5148RGYR"
+			(at 172.72 109.22 0)
+			(effects
+				(font
+					(size 1.27 1.27)
+				)
+				(justify left)
+				(hide yes)
+			)
+		)
+		(property "Mouser Part Number" "595-LM5148RGYR"
+			(at 172.72 111.76 0)
+			(effects
+				(font
+					(size 1.27 1.27)
+				)
+				(justify left)
+				(hide yes)
+			)
+		)
+		(property "Mouser Price/Stock" "https://www.mouser.co.uk/ProductDetail/Texas-Instruments/LM5148RGYR?qs=Jm2GQyTW%2FbgsJOyzcNbTmw%3D%3D"
+			(at 172.72 114.3 0)
+			(effects
+				(font
+					(size 1.27 1.27)
+				)
+				(justify left)
+				(hide yes)
+			)
+		)
+		(property "Arrow Part Number" "LM5148RGYR"
+			(at 172.72 116.84 0)
+			(effects
+				(font
+					(size 1.27 1.27)
+				)
+				(justify left)
+				(hide yes)
+			)
+		)
+		(property "Arrow Price/Stock" "https://www.arrow.com/en/products/lm5148rgyr/texas-instruments?region=nac"
+			(at 172.72 119.38 0)
+			(effects
+				(font
+					(size 1.27 1.27)
+				)
+				(justify left)
+				(hide yes)
+			)
+		)
+		(pin "19"
+		)
+		(pin "12"
+		)
+		(pin "4"
+		)
+		(pin "16"
+		)
+		(pin "18"
+		)
+		(pin "6"
+		)
+		(pin "9"
+		)
+		(pin "17"
+		)
+		(pin "5"
+		)
+		(pin "3"
+		)
+		(pin "2"
+		)
+		(pin "15"
+		)
+		(pin "13"
+		)
+		(pin "14"
+		)
+		(pin "11"
+		)
+		(pin "21"
+		)
+		(pin "8"
+		)
+		(pin "25"
+		)
+		(pin "1"
+		)
+		(pin "20"
+		)
+		(pin "23"
+		)
+		(pin "10"
+		)
+		(pin "22"
+		)
+		(pin "7"
+		)
+		(pin "24"
+		)
+		(instances
+			(project ""
+				(path "/2b20bf84-f1a7-4c48-aa1b-8d85c83ac6e5"
+					(reference "IC1")
+					(unit 1)
+				)
+			)
+		)
 	)
 	(symbol
@@
 					(unit 1)
 				)
-			)
-		)
-	)
-	(symbol
-		(lib_name "LM5148RGYR_1")
-		(lib_id "LM5148RGYR_edited normal_symbol:LM5148RGYR")
-		(at 123.19 95.25 0)
-		(unit 1)
-		(exclude_from_sim no)
-		(in_bom yes)
-		(on_board yes)
-		(dnp no)
-		(fields_autoplaced yes)
-		(property "Reference" "IC3"
-			(at 143.51 77.47 0)
-			(effects
-				(font
-					(size 1.27 1.27)
-				)
-			)
-		)
-		(property "Value" "LM5148RGYR"
-			(at 143.51 80.01 0)
-			(effects
-				(font
-					(size 1.27 1.27)
-				)
-			)
-		)
-		(property "Footprint" "LM5148_:LM5148RGYR"
-			(at 138.176 84.074 0)
-			(effects
-				(font
-					(size 1.27 1.27)
-				)
-				(justify left)
-				(hide yes)
-			)
-		)
-		(property "Datasheet" "https://www.ti.com/lit/ds/symlink/lm5148.pdf?ts=1680990210570&ref_url=https%253A%252F%252Fwww.ti.com%252Fproduct%252FLM5148"
-			(at 171.958 74.676 0)
-			(effects
-				(font
-					(size 1.27 1.27)
-				)
-				(justify left)
-				(hide yes)
-			)
-		)
-		(property "Description" "Switching Controllers 3.5-V to 80-V, current mode synchronous buck controller"
-			(at 100.33 116.84 0)
-			(effects
-				(font
-					(size 1.27 1.27)
-				)
-				(hide yes)
-			)
-		)
-		(property "Description_1" "Switching Controllers 3.5-V to 80-V, current mode synchronous buck controller"
-			(at 171.958 77.216 0)
-			(effects
-				(font
-					(size 1.27 1.27)
-				)
-				(justify left)
-				(hide yes)
-			)
-		)
-		(property "Height" "1"
-			(at 160.02 90.17 0)
-			(effects
-				(font
-					(size 1.27 1.27)
-				)
-				(justify left)
-				(hide yes)
-			)
-		)
-		(property "Manufacturer_Name" "Texas Instruments"
-			(at 172.72 106.68 0)
-			(effects
-				(font
-					(size 1.27 1.27)
-				)
-				(justify left)
-				(hide yes)
-			)
-		)
-		(property "Manufacturer_Part_Number" "LM5148RGYR"
-			(at 172.72 109.22 0)
-			(effects
-				(font
-					(size 1.27 1.27)
-				)
-				(justify left)
-				(hide yes)
-			)
-		)
-		(property "Mouser Part Number" "595-LM5148RGYR"
-			(at 172.72 111.76 0)
-			(effects
-				(font
-					(size 1.27 1.27)
-				)
-				(justify left)
-				(hide yes)
-			)
-		)
-		(property "Mouser Price/Stock" "https://www.mouser.co.uk/ProductDetail/Texas-Instruments/LM5148RGYR?qs=Jm2GQyTW%2FbgsJOyzcNbTmw%3D%3D"
-			(at 172.72 114.3 0)
-			(effects
-				(font
-					(size 1.27 1.27)
-				)
-				(justify left)
-				(hide yes)
-			)
-		)
-		(property "Arrow Part Number" "LM5148RGYR"
-			(at 172.72 116.84 0)
-			(effects
-				(font
-					(size 1.27 1.27)
-				)
-				(justify left)
-				(hide yes)
-			)
-		)
-		(property "Arrow Price/Stock" "https://www.arrow.com/en/products/lm5148rgyr/texas-instruments?region=nac"
-			(at 172.72 119.38 0)
-			(effects
-				(font
-					(size 1.27 1.27)
-				)
-				(justify left)
-				(hide yes)
-			)
-		)
-		(pin "18"
-		)
-		(pin "19"
-		)
-		(pin "3"
-		)
-		(pin "2"
-		)
-		(pin "6"
-		)
-		(pin "9"
-		)
-		(pin "17"
-		)
-		(pin "12"
-		)
-		(pin "5"
-		)
-		(pin "13"
-		)
-		(pin "11"
-		)
-		(pin "15"
-		)
-		(pin "14"
-		)
-		(pin "24"
-		)
-		(pin "20"
-		)
-		(pin "23"
-		)
-		(pin "8"
-		)
-		(pin "25"
-		)
-		(pin "10"
-		)
-		(pin "7"
-		)
-		(pin "4"
-		)
-		(pin "1"
-		)
-		(pin "21"
-		)
-		(pin "16"
-		)
-		(pin "22"
-		)
-		(instances
-			(project ""
-				(path "/2b20bf84-f1a7-4c48-aa1b-8d85c83ac6e5"
-					(reference "IC3")
-					(unit 1)
-				)

Commit message: final updates
straight polygons, straight tracks, Proper ERC, corrected the unrouted tracks
Other:
- note added: "I/O Pads"
- note added: "Mounting Holes"
- note added: "Net-tie"
